File: hardware/kicad/bwlr1f.kicad_sch (KiCad schematic)
At the start: 66 parts, among them J1 Conn_01x02, Q2 PMV32UP, Q3 DMG1012UW, U1 BME688, U1 RAK3172-SIP, U2 NBM7100ABQX, U3 ZD24C08A, U5 TPL5110

Commit message: first production file revision 1
Parts:
- removed C10, C3 (x7): 100nF, Capacitor_SMD:C_0402_1005Metric, symbol Device:C_Small
- removed C3 (x5): 1uF, Capacitor_SMD:C_0402_1005Metric, symbol Device:C_Small
- removed C3: 4.7uF, Capacitor_SMD:C_0402_1005Metric, symbol Device:C_Small
- removed Q2: PMV32UP, Package_TO_SOT_SMD:SOT-23, symbol Simulation_SPICE:PMOS
- removed R11: 100K, Resistor_SMD:R_0402_1005Metric, symbol Device:R_Small
- removed R11: 1M, Resistor_SMD:R_0402_1005Metric, symbol Device:R_Small
- removed R4: 1K, Resistor_SMD:R_0402_1005Metric, symbol Device:R_Small
- removed R5: 4.7K, Resistor_SMD:R_0402_1005Metric, symbol Device:R_Small
- removed R5 (x2): 10K, Resistor_SMD:R_0402_1005Metric, symbol Device:R_Small
- added BT2: Battery_Cell, bwlr1f:BAT-SMD_MY-2032-12, symbol Device:Battery_Cell
- added C3 (x8): 100n, Capacitor_SMD:C_0402_1005Metric, symbol Device:C_Small
- added C3 (x4): 1u, Capacitor_SMD:C_0402_1005Metric, symbol Device:C_Small
- added C3 (x2): 4u7, Capacitor_SMD:C_0402_1005Metric, symbol Device:C_Small
- added Q2: PMV32UP, Package_TO_SOT_SMD:SOT-23, symbol Device:Q_PMOS_GSD
- added R11: 100K, Resistor_SMD:R_0402_1005Metric, symbol Device:R_Small
- added R16: 1M, Resistor_SMD:R_0402_1005Metric, symbol Device:R_Small
- added R3 (x2): 10K, Resistor_SMD:R_0402_1005Metric, symbol Device:R_Small
- added R4: 1K, Resistor_SMD:R_0402_1005Metric, symbol Device:R_Small
- added R4: 4K7, Resistor_SMD:R_0402_1005Metric, symbol Device:R_Small
- added TP1: BATT+, TestPoint:TestPoint_Pad_D1.0mm, symbol Connector:TestPoint
- BT1: Distributor (none) -> LCSC; Distributor Link (none) -> https://www.lcsc.com/product-detail/Battery-Connectors_MYOU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; Distributor Part Number (none) -> C964833; Manufacturer (none) -> MYOUNG; Manufacturer Part Number (none) -> MY-2032-12; Part Description (none) -> Battery button -25℃~+85℃ CR2032
- C16: value 470uF -> 470u; Distributor (none) -> Digikey; Distributor Link (none) -> https://www.digikey.com/en/products/detail/kyocera-avx/TCJ5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; Distributor Part Number (none) -> 478-13191-1-ND; Part Description (none) -> Tantalum Polymer Capacitor 470 µF 16V 100mOhm @ 100kHz
- C3: value 22uF -> 22u; Distributor (none) -> LCSC; Distributor Link (none) -> https://www.lcsc.com/product-detail/Multilayer-Ceramic-Capa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; Distributor Part Number (none) -> C7472972; Part Description 16V, X7R, <10% -> Ceramic Capacitors 16V 22uF X7R ±10%
- C3, C5: value 100nF -> 100n; Distributor (none) -> LCSC; Distributor Link (none) -> https://www.lcsc.com/product-detail/Multilayer-Ceramic-Capa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; Distributor Part Number (none) -> C1525; Part Description Ceramic Capacitor 100nF 10% 10V X7R -> Ceramic Capacitor 100nF 10% 16V X7R
- C3: value 1uF -> 1u; Distributor (none) -> LCSC; Distributor Link (none) -> https://www.lcsc.com/product-detail/Multilayer-Ceramic-Capa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; Distributor Part Number (none) -> C29266; Part Description (none) -> Ceramic Capacitors 16V 1uF X5R ±10%
- C3: value 1uF -> 1u; Distributor (none) -> LCSC; Distributor Link (none) -> https://www.lcsc.com/product-detail/Multilayer-Ceramic-Capa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; Distributor Part Number (none) -> C29266; Part Description (none) -> Multilayer Ceramic Capacitors 16V 1uF X5R ±10%
- C3: value 470nF -> 470n; Distributor (none) -> LCSC; Distributor Link (none) -> https://www.lcsc.com/product-detail/Multilayer-Ceramic-Capa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; Distributor Part Number (none) -> C47339; Part Description (none) -> Ceramic Capacitors 10V 470nF X5R ±10%
- C3: value 10uF -> 10u; Distributor (none) -> LCSC; Distributor Link (none) -> https://www.lcsc.com/product-detail/Multilayer-Ceramic-Capa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; Distributor Part Number (none) -> C962136; Part Description (none) -> Ceramic Capacitors 16V 10uF X5R ±10%
- C3: value 4.7uF -> 4u7; Distributor (none) -> LCSC; Distributor Link (none) -> https://www.lcsc.com/product-detail/Multilayer-Ceramic-Capa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; Distributor Part Number (none) -> C368809; Part Description (none) -> Ceramic Capacitors 10V 4.7uF X5R ±10%
- E1: Distributor (none) -> Digikey; Distributor Link (none) -> https://www.digikey.com/en/products/detail/te-connectivity-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; Distributor Part Number (none) -> 343-ANT-915-USP410CT-ND; MANUFACTURER Linx -> (none); MAXIMUM_PACKAGE_HEIGHT 2.9 mm -> (none); Manufacturer (none) -> TE Connectivity Linx; Manufacturer Part Number (none) -> ANT-915-USP410; PARTREV N/A -> (none); Part Description (none) -> 915MHz ISM, LoRaWAN, LPWA, Sigfox Chip RF Antenna 902MHz ~ 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; STANDARD Manufacturer Recommendations -> (none)
- L1: Distributor (none) -> LCSC; Distributor Link (none) -> https://www.lcsc.com/product-detail/Chip-Resistor-Surface-M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; Distributor Part Number (none) -> C21189; Manufacturer (none) -> UNI-ROYAL(Uniroyal Elec); Manufacturer Part Number (none) -> 0603WAF0000T5E; Part Description (none) -> Resistors 100mW 75V ±1% 0Ω
- L1, L3, L4: footprint Inductor_SMD:L_0603_1608Metric -> Inductor_SMD:L_0402_1005Metric; Distributor (none) -> LCSC; Distributor Link (none) -> https://www.lcsc.com/product-detail/Ferrite-Beads_Murata-El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; Distributor Part Number (none) -> C76891; Manufacturer Sunlord -> Murata Electronics; Manufacturer Part Number MZAS1608G121-1R3TF -> BLM15PD121SN1D; Part Description (none) -> Ferrite Beads 90mΩ ±25% 120Ω@100MHz
- L2: value 15uH -> 15u; Distributor (none) -> LCSC; Distributor Link (none) -> https://www.lcsc.com/product-detail/Inductors-SMD_TDK-MLZ20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; Distributor Part Number (none) -> C383402; Part Description (none) -> Inductors 15uH ±20% 120mA 950mΩ
- L2: value 15uH -> 15u; Distributor (none) -> Digikey; Distributor Link (none) -> https://www.digikey.com/en/products/detail/w%C3%BCrth-elekt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; Distributor Part Number (none) -> 732-5509-1-ND; Part Description (none) -> Wirewound Inductor 15 µH Semi-Shielded Drum Core, 850 mA 21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
- R10: value 16.9K -> 16K9; Distributor (none) -> LCSC; Distributor Link (none) -> https://www.lcsc.com/product-detail/Chip-Resistor-Surface-M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; Distributor Part Number (none) -> C163488; Part Description (none) -> Resistors 62.5mW 50V ±100ppm/℃ ±1% 16.9kΩ
- R11: Distributor (none) -> LCSC; Distributor Link (none) -> https://www.lcsc.com/product-detail/Chip-Resistor-Surface-M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; Distributor Part Number (none) -> C60491; Part Description (none) -> Resistors 62.5mW 50V ±100ppm/℃ ±1% 100kΩ
- R2, R3: Distributor (none) -> LCSC; Distributor Link (none) -> https://www.lcsc.com/product-detail/Chip-Resistor-Surface-M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; Distributor Part Number (none) -> C60490; Part Description Resistor 10K 5% 100mW -> Resistor 10K 1% 62.5mW
- R4: value 4.7K -> 4K7; Distributor (none) -> LCSC; Distributor Link (none) -> https://www.lcsc.com/product-detail/Chip-Resistor-Surface-M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; Distributor Part Number (none) -> C105871; Part Description (none) -> Resistor 62.5mW 50V ±100ppm/℃ ±1% 4.7kΩ
- R4: Distributor (none) -> LCSC; Distributor Link (none) -> https://www.lcsc.com/product-detail/Chip-Resistor-Surface-M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; Distributor Part Number (none) -> C106235; Part Description (none) -> Resistors 62.5mW 50V ±100ppm/℃ ±1% 1kΩ
- U1: Distributor (none) -> RAKwireless; Distributor Link (none) -> Contact inquiry@rakwireless.com for SKU: 306039; Distributor Part Number (none) -> 306039; Manufacturer (none) -> RAKwireless; Manufacturer Part Number (none) -> 306039; Part Description (none) -> Low Power STM32WLE5 Module for LoRaWAN
- U1: Distributor (none) -> Digikey; Distributor Link (none) -> https://www.digikey.com/en/products/detail/bosch-sensortec/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; Distributor Part Number (none) -> 828-BME688CT-ND; Part Description (none) -> Gas, Humidity, Pressure, Temperature Sensor I²C, SPI Output
- U2: Distributor (none) -> Digikey; Distributor Link (none) -> https://www.digikey.com/en/products/detail/nexperia-usa-inc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; Distributor Part Number (none) -> 1727-NBM7100ABQXCT-ND; Part Description (none) -> Coin cell battery life booster
- U3: Distributor (none) -> LCSC; Distributor Link (none) -> https://www.lcsc.com/product-detail/EEPROM_Zetta-ZD24C08A-S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; Distributor Part Number (none) -> C2896640; Part Description (none) -> 8Kbit 1MHz I2C SOT-23-5 EEPROM
- U5: Distributor (none) -> LCSC; Distributor Link (none) -> https://www.lcsc.com/product-detail/Timers-Clock-Oscillator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; Distributor Part Number (none) -> C125830; Manufacturer (none) -> Texas Instruments; Manufacturer Part Number (none) -> TPL5110DDCT; Part Description (none) -> Timers / Clock Oscillators
Connections:
- net +3V0: now also C3.2, C3.2, C3.2, C3.2, C3.2, C3.2, Q2.3 (D), R3.1, R4.1
- net +VDP: now also C3.2, R4.1
- net BATT+: now also BT2.1 (+), C3.2, C3.2, TP1.1
- net BOOT: now also R3.1
- net DONE: now also R16.1
- net DRV: now also Q2.1 (G)
- net GND: now also BT2.2 (-), C3.1, C3.1, C3.1, C3.1, C3.1, C3.1, C3.1, C3.1, C3.1, C3.1, C3.1, C3.1, C3.1, C3.1, R11.2, R16.2, R3.2
- net RST: now also C3.2, R3.2
- net SDA: now also R4.2, R4.2
- net at C3.2, L2.1, U1.10 (VFBSMPS): now also C3.2
- net at L4.1, U1.53 (VDDPA): now also C3.2
- net at U2.4 (ADR): now also R11.1
- net at L1.2, U1.11 (VDDMPS): now also C3.2
- net at JP1.2 (C): now also Q2.2 (S)
- net at L3.1, U1.54 (VDDRF): now also C3.2
Other:
- note added: "Antenna"
- note added: "Battery Input"
- note added: "Connectors"
- note added: "Coplanar Waveguide with Ground Characteristic"
- note added: "Effective Dielectric Constant: 3.188 Characteristic Impedance: 50.15ohm"
- note added: "Environmental Sensor"
- note added: "I2C Address: 0x77"
- note added: "Main Controller"
- note added: "NV Storage"
- note added: "Power Gate"
- note added: "Power Gating Time Interval: +/- 30s"
- note added: "Power Regulator"
- note added: "Programming Port"
- note added: "Relative Dielectric Constant: 4.29 Track Width : 0.21mm Gap Width : 0.15mm Dielectric Thickness : 0.11mm"
- note removed: "+/- 30s"
- note removed: "16V, ceramic, low esr"
- note removed: "ANTENNA"
- note removed: "BME688 Environmental Sensor"
- note removed: "CONNECTORS"
- note removed: "Coplanar Waveguide With Ground Characteristic"
- note removed: "EEPROM"
- note removed: "Effective Dielectric Constant: 2.33 Characteristic Impedance: 50.19ohm"
- note removed: "NBM7100A"
- note removed: "Power Gating Time Interval:"
- note removed: "RAK3172-SIP"
- note removed: "Relative Dielectric Constant: 4.5 Track Width : 0.8mm Gap Width : 0.15mm Dielectric Thickness : 1.6mm"
- note removed: "TPL5110"
- note removed: "wurth 74404042150"
- title: BWLR1F -> Teapotlabs BWLR1F
- moved on the sheet: BT1, C15, C16, C3, E1, J1, JP1, L1, L2, R11, R4, TP1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

Commit message: add initial mdrv latcher circuit
Parts:
- removed Q2: PMV32UP, Package_TO_SOT_SMD:SOT-23, symbol Device:Q_PMOS_GSD
- removed R16 (x2): 1M, Resistor_SMD:R_0402_1005Metric, symbol Device:R_Small
- added C3: 100n, Capacitor_SMD:C_0402_1005Metric, symbol Device:C_Small
- added Q2 (x2): PMV32UP, Package_TO_SOT_SMD:SOT-23, symbol Device:Q_PMOS_GSD
- added R10: 22K, Resistor_SMD:R_0402_1005Metric, symbol Device:R_Small
- added R16 (x3): 1M, Resistor_SMD:R_0402_1005Metric, symbol Device:R_Small
- added U6: TPL5110, Package_TO_SOT_SMD:SOT-23-6, symbol Timer:TPL5110
Connections:
- net BATT+: now also C3.2, Q2.2 (S), Q2.2 (S), R16.1, U6.1 (VDD)
- net DELAY_MDRV: now also R16.1; no longer TP6.1
- net GND: now also C3.1, R10.2, R16.2, R16.2, U6.2 (GND), U6.6 (EN/ONE_SHOT)
- net at Q3.3 (D): now also Q2.1 (G), R16.2
- net DELAY_MDRV_IN: now reaches R10.1, U5.3 (DELAY/M_DRV)
- net DELAY_MDRV_IN: now also TP6.1, Q2.3 (D)
- net MDL_DONE: now reaches U1.24 (PC3)
- net MDL_DONE: now also R16.1, U6.4 (DONE)
- new net: Q2.1 (G), U6.5 (DRV)
- new net: Q2.3 (D), R10.1, U6.3 (DELAY/M_DRV)
- no-connect marks 27 -> 26
Other:
- note added: "MCU Power Gate"
- note added: "Power Gate MDRV Latcher"
- note added: "Power Gating Time Interval: +/- 1m"
- note removed: "Power Gate"
- moved on the sheet: C3, R10, R16, U5
