File: hardware/main/kicad/bwlr1f.kicad_sch (KiCad schematic)
At the start: 68 parts, among them J1 Conn_01x02, U1 BME688, U1 RAK3172-SIP, U2 NBM7100ABQX, U3 ZD24C08A, U5 RV-3028-C7

Commit message: Change PCB Antenna
Parts:
- removed E1: ANT-915-USP410, bwlr1f:XDCR_ANT-915-USP410, symbol bwlr1f:ANT-915-USP410
- added AE1: Antenna, RF_Antenna:Texas_SWRA416_868MHz_915MHz, symbol Device:Antenna
Connections:
- net ANT: now also AE1.1 (A)
Other:
- moved on the sheet: R4

Commit message: Revert "Change PCB Antenna"
This reverts commit 5ca8b7b7452485b6d3384e8d9324ab527cbc9679.
Parts:
- removed AE1: Antenna, RF_Antenna:Texas_SWRA416_868MHz_915MHz, symbol Device:Antenna
- added E1: ANT-915-USP410, bwlr1f:XDCR_ANT-915-USP410, symbol bwlr1f:ANT-915-USP410
Connections:
- net ANT: now also E1.1
- net GND: now also E1.2
Other:
- moved on the sheet: R4

Commit message: Revision finish, update production file
Parts:
- removed E1: ANT-915-USP410, bwlr1f:XDCR_ANT-915-USP410, symbol bwlr1f:ANT-915-USP410
- added AE1: Antenna, RF_Antenna:Texas_SWRA416_868MHz_915MHz, symbol Device:Antenna
Connections:
- net ANT: now also AE1.1 (A)
Other:
- note removed: "Coplanar Waveguide with Ground Characteristic"
- note removed: "Effective Dielectric Constant: 3.188 Characteristic Impedance: 50.15ohm"
- note removed: "Relative Dielectric Constant: 4.29 Track Width : 0.21mm Gap Width : 0.15mm Dielectric Thickness : 0.11mm"
- note removed: "Trace characteristics"
- moved on the sheet: C15, C16, L1
