File: hardware/main/kicad/bwlr1f.kicad_sch (KiCad schematic)
At the start: 60 parts, among them J1 Conn_01x02, U1 BME688, U1 RAK3172-SIP, U2 NBM7100ABQX, U3 ZD24C08A, U5 RV-3028-C7

Commit message: Update Programmer
Connections:
- net RTC_WKUP: now also U1.14 (PB3); no longer U1.5 (PC13)
Changed lines of the file:
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@@
 	)
 	(no_connect
-		(at 82.55 127)
+		(at 82.55 99.06)
 	)
 	(no_connect
@@
 	(wire
 		(pts
-			(xy 72.39 99.06) (xy 82.55 99.06)
-		)
-		(stroke
-			(width 0)
-			(type default)
-		)
-	)
-	(wire
-		(pts
 			(xy 163.83 104.14) (xy 163.83 102.87)
 		)
@@
 		(pts
 			(xy 129.54 81.28) (xy 129.54 76.2)
+		)
+		(stroke
+			(width 0)
+			(type default)
+		)
+	)
+	(wire
+		(pts
+			(xy 72.39 127) (xy 82.55 127)
 		)
 		(stroke
@@
 	)
 	(label "RTC_WKUP"
-		(at 72.39 99.06 0)
-		(fields_autoplaced yes)
-		(effects
+		(at 72.39 127 0)
+		(fields_autoplaced yes)
+		(effects

Commit message: Added ESD to main board
Parts:
- added D1, D2, D3, D4, D5, D6, D7, D8: ESD5651N, Diode_SMD:D_SOD-882, symbol Device:D_TVS
Connections:
- net +3V0: now also D8.2 (A2)
- net BATT+: now also D7.2 (A2)
- net BOOT: now also D1.2 (A2)
- net GND: now also D1.1 (A1), D2.1 (A1), D3.1 (A1), D4.1 (A1), D5.1 (A1), D6.1 (A1), D7.1 (A1), D8.1 (A1)
- net RST: now also D2.2 (A2)
- net RX2: now also D6.2 (A2)
- net SWCLK: now also D4.2 (A2)
- net SWDIO: now also D3.2 (A2)
- net TX2: now also D5.2 (A2)
Other:
- note added: "Battery"
- note removed: "Battery Input"
- note removed: "Connectors"
- note removed: "Uart brigde > Level translator"
- moved on the sheet: BT1, BT2, C15, C16, C3, E1, J1, JP1, L1, L2, R11, R4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

Commit message: Finish Production File for Main Board
Parts:
- BT1, BT2, C16, C24, C3, C5, E1, L1, L2, L3, L4, R11, R2, R3, R4, U1, U2, U3: Type (none) -> SMT
- C15, C16, J1, JP1: Distributor (none) -> -; Distributor Link (none) -> -; Distributor Part Number (none) -> -; Manufacturer (none) -> -; Manufacturer Part Number (none) -> -; Type (none) -> SMT
- D1, D2, D3, D4, D5, D6, D7, D8: Type SMD -> SMT
- TP1: value BATT+ -> ProgPin; Distributor (none) -> -; Distributor Link (none) -> -; Distributor Part Number (none) -> -; Manufacturer (none) -> -; Manufacturer Part Number (none) -> -; Type (none) -> SMT
- TP1: value RX2 -> ProgPin; Distributor (none) -> -; Distributor Link (none) -> -; Distributor Part Number (none) -> -; Manufacturer (none) -> -; Manufacturer Part Number (none) -> -; Type (none) -> SMT
- TP2: value TX2 -> ProgPin; Distributor (none) -> -; Distributor Link (none) -> -; Distributor Part Number (none) -> -; Manufacturer (none) -> -; Manufacturer Part Number (none) -> -; Type (none) -> SMT
- TP3: value SWCLK -> ProgPin; Distributor (none) -> -; Distributor Link (none) -> -; Distributor Part Number (none) -> -; Manufacturer (none) -> -; Manufacturer Part Number (none) -> -; Type (none) -> SMT
- TP4: value SWDIO -> ProgPin; Distributor (none) -> -; Distributor Link (none) -> -; Distributor Part Number (none) -> -; Manufacturer (none) -> -; Manufacturer Part Number (none) -> -; Type (none) -> SMT
- TP5: value RST -> ProgPin; Distributor (none) -> -; Distributor Link (none) -> -; Distributor Part Number (none) -> -; Manufacturer (none) -> -; Manufacturer Part Number (none) -> -; Type (none) -> SMT
- TP6: value BOOT -> ProgPin; Distributor (none) -> -; Distributor Link (none) -> -; Distributor Part Number (none) -> -; Manufacturer (none) -> -; Manufacturer Part Number (none) -> -; Type (none) -> SMT
- TP8: value GND -> ProgPin; Distributor (none) -> -; Distributor Link (none) -> -; Distributor Part Number (none) -> -; Manufacturer (none) -> -; Manufacturer Part Number (none) -> -; Type (none) -> SMT
- TP8: value 3V0 -> ProgPin; Distributor (none) -> -; Distributor Link (none) -> -; Distributor Part Number (none) -> -; Manufacturer (none) -> -; Manufacturer Part Number (none) -> -; Type (none) -> SMT
- U5: Distributor (none) -> LCSC; Distributor Link (none) -> https://www.lcsc.com/product-detail/Real-Time-Clocks_Micro-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; Distributor Part Number (none) -> C3019759; Manufacturer (none) -> Micro Crystal; Manufacturer Part Number (none) -> RV-3028-C7 32.768kHz 1ppm TA QC; Type (none) -> SMT
