File: hardware/main/kicad/bwlr1f.kicad_pcb (KiCad board)
At the start: 4 copper layers, 63.5 x 26.1 mm, 69 parts, among them J1 Conn_01x02, U1 RAK3172-SIP, U2 NBM7100ABQX, U3 ZD24C08A, U4 BME688, U5 RV-3028-C7

Commit message: update silkscreen rev identifier
Other:
- board text added: "Typ. A Rev. 2"
- board text removed: "Rev. A 08/24"
Changed lines of the file:
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@@
 		(layer "Edge.Cuts")
 	)
-	(gr_text "Rev. A   08/24"
+	(gr_text "Typ. A   Rev. 2"
 		(at 154.364999 119.191 0)
 		(layer "B.SilkS")
