File: hardware/main/kicad/bwlr1f.kicad_pcb (KiCad board)
At the start: 4 copper layers, 61.2 x 26.1 mm, 69 parts, among them J1 Conn_01x02, U1 RAK3172-SIP, U2 NBM7100ABQX, U3 ZD24C08A, U4 BME688, U5 RV-3028-C7

Commit message: Change PCB Antenna
Parts:
- removed E1: ANT-915-USP410, bwlr1f:XDCR_ANT-915-USP410
- added AE1: Antenna, RF_Antenna:Texas_SWRA416_868MHz_915MHz, F.Cu at (161.5, 110.6)
- C22, C23, C25, R1, R11, R2: moved to B.Cu
- moved G*** 36.8 mm to (125.0, 140.0)
- moved R11 26.1 mm to (128.1, 101.8)
- moved C22 23.9 mm to (129.1, 101.8)
- moved U4 22.8 mm to (129.3, 102.5), turned to -90 degrees
- moved C23 20.8 mm to (130.6, 101.8), turned to 90 degrees
- moved R12 17.9 mm to (131.6, 101.8), turned to -90 degrees
- moved C20 8.71 mm to (153.5, 101.5), turned to 0 degrees
- moved R1 7.39 mm to (142.2, 103.7)
- moved R2 7.39 mm to (141.2, 103.7)
- moved C25 6.11 mm to (128.1, 107.1), turned to 90 degrees
- moved L6 5.90 mm to (154.2, 103.8), turned to 90 degrees
- moved C18 5.43 mm to (153.5, 106.1), turned to 0 degrees
- moved U5 5.11 mm to (129.3, 111.8), turned to 90 degrees
- moved U3 4.73 mm to (129.3, 107.1), turned to 180 degrees
- moved R3 3.00 mm to (150.3, 103.7), turned to 90 degrees
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Routing:
- net /SDA: track 60.8 -> 40.5 mm, vias 5 -> 6
- net +3V0: track 53.2 -> 35.8 mm, vias 11 -> 13
- net /RTC_WKUP: track 15.2 -> 0.00 mm, vias 2 -> 0
- net /RST: track 21.8 -> 7.82 mm, vias 2 -> 1
- net /SCL: track 59.0 -> 46.6 mm
- net /BOOT: track 19.1 -> 9.13 mm, vias 2 -> 1
- net GND: track 32.4 -> 22.6 mm, vias 102 -> 77
- net /RF: track 3.44 -> 11.3 mm
- net Net-(JP1-B): track 5.41 -> 0.00 mm, vias 2 -> 0
- net /SWCLK: track 24.4 -> 21.7 mm
- net /SWDIO: track 23.4 -> 21.6 mm
- net /RX2: track 9.21 -> 7.46 mm
- net /START: track 5.39 -> 3.85 mm
- net Net-(U4-SDO): track 1.44 -> 0.00 mm
- net /RDY: track 5.81 -> 4.46 mm
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Other:
- board size 61.2 x 26.1 mm -> 64.1 x 26.1 mm

Commit message: Revert "Change PCB Antenna"
This reverts commit 5ca8b7b7452485b6d3384e8d9324ab527cbc9679.
Parts:
- removed AE1: Antenna, RF_Antenna:Texas_SWRA416_868MHz_915MHz
- added E1: ANT-915-USP410, bwlr1f:XDCR_ANT-915-USP410, F.Cu at (161.6, 114.5)
- C22, C23, C25, R1, R11, R2: moved to F.Cu
- moved G*** 36.8 mm to (152.0, 114.9)
- moved R11 26.1 mm to (153.9, 105.5)
- moved C22 23.9 mm to (152.7, 105.5)
- moved U4 22.8 mm to (152.1, 102.6), turned to 90 degrees
- moved C23 20.8 mm to (151.2, 105.0), turned to 180 degrees
- moved R12 17.9 mm to (149.6, 101.9), turned to 90 degrees
- moved C20 8.71 mm to (154.7, 110.2), turned to 90 degrees
- moved R1 7.39 mm to (135.2, 101.3)
- moved R2 7.39 mm to (134.2, 101.3)
- moved C25 6.11 mm to (132.5, 102.9), turned to -90 degrees
- moved L6 5.90 mm to (152.3, 109.4), turned to 0 degrees
- moved C18 5.43 mm to (149.9, 110.2), turned to 90 degrees
- moved U5 5.11 mm to (129.9, 106.7), turned to -90 degrees
- moved U3 4.73 mm to (129.9, 102.4), turned to 0 degrees
- moved R3 3.00 mm to (147.9, 105.5), turned to 180 degrees
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Routing:
- net /SDA: track 40.5 -> 60.8 mm, vias 6 -> 5
- net +3V0: track 35.8 -> 53.2 mm, vias 13 -> 11
- net /RTC_WKUP: track 0.00 -> 15.2 mm, vias 0 -> 2
- net /RST: track 7.82 -> 21.8 mm, vias 1 -> 2
- net /SCL: track 46.6 -> 59.0 mm
- net /BOOT: track 9.13 -> 19.1 mm, vias 1 -> 2
- net GND: track 22.6 -> 32.4 mm, vias 77 -> 102
- net /RF: track 11.3 -> 3.44 mm
- net Net-(JP1-B): track 0.00 -> 5.41 mm, vias 0 -> 2
- net /SWCLK: track 21.7 -> 24.4 mm
- net /SWDIO: track 21.6 -> 23.4 mm
- net /RX2: track 7.46 -> 9.21 mm
- net /START: track 3.85 -> 5.39 mm
- net Net-(U4-SDO): track 0.00 -> 1.44 mm
- net /RDY: track 4.46 -> 5.81 mm
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Other:
- board size 64.1 x 26.1 mm -> 61.2 x 26.1 mm

Commit message: clean-up
Routing:
- net GND: track 32.4 -> 34.1 mm
Other:
- board text added: "Typ. B Rev. 2"
- board text removed: "Rev. A 08/24"
Changed lines of the file:
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@@
 	(title_block
 		(title "Teapotlabs BWLR1F")
-		(date "2024-01-09")
-		(rev "1")
+		(date "2024-08-27")
+		(rev "2")
 		(company "Teapot Laboratories")
 	)
@@
 		(layer "Edge.Cuts")
 	)
-	(gr_text "Rev. A   08/24"
+	(gr_text "Typ. B   Rev. 2"
 		(at 154.491999 117.667 0)
 		(layer "B.SilkS")
@@
 		)
 		(height -4.004152)
-		(gr_text "889,4383 mils"
+		(gr_text "22.5917 mm"
 			(at 171.001999 110.555 90)
 			(layer "User.2")
@@
 		)
 		(height -16.394027)
-		(gr_text "2410,7272 mils"
+		(gr_text "61.2325 mm"
 			(at 136.085662 93.009973 0.001871418142)
 			(layer "User.2")
@@
 		)
 		(height 5.447999)
-		(gr_text "1028,7402 mils"
+		(gr_text "26.1300 mm"
 			(at 101.272 110.555 90)
 			(layer "User.2")
@@
 	)
 	(segment
-		(start 129.599999 102.427)
-		(end 128.716499 102.427)
-		(width 0.25)
+		(start 155.569999 118.6095)
+		(end 155.569999 120.5505)
+		(width 0.5)
 		(layer "F.Cu")
 		(net 1)
 	)
 	(segment
-		(start 142.631847 100.343248)
-		(end 142.631847 101.578)
+		(start 129.599999 102.427)
+		(end 128.716499 102.427)
 		(width 0.25)
 		(layer "F.Cu")
@@
 	)
 	(segment
-		(start 156.763999 119.558)
-		(end 155.507999 118.302)
+		(start 142.631847 100.343248)
+		(end 142.631847 101.578)
 		(width 0.25)
 		(layer "F.Cu")
@@
 	)
 	(segment
-		(start 156.791999 119.558)
-		(end 155.507999 120.842)
-		(width 0.25)
-		(layer "F.Cu")
-		(net 1)
-	)
-	(segment
-		(start 157.053999 119.558)
-		(end 156.763999 119.558)
-		(width 0.25)
-		(layer "F.Cu")
-		(net 1)
-	)
-	(segment
 		(start 134.270999 105.884)
 		(end 133.790999 105.884)
@@
 	)
 	(segment
-		(start 157.053999 119.558)
-		(end 156.791999 119.558)
-		(width 0.25)
-		(layer "F.Cu")
-		(net 1)
-	)
-	(segment
 		(start 147.125999 110.588)
 		(end 148.041847 110.588)
@@
 	)
 	(segment
+		(start 155.559999 118.335)
+		(end 155.559999 120.276)
+		(width 0.5)
+		(layer "F.Cu")
+		(net 1)
+	)
+	(segment
 		(start 144.431847 111.952)
 		(end 144.431847 112.878)
@@
 	)
 	(segment
+		(start 155.559999 118.874)
+		(end 155.559999 120.815)
+		(width 0.5)
+		(layer "F.Cu")
+		(net 1)
+	)
+	(segment
 		(start 142.556599 100.268)
 		(end 142.631847 100.343248)
@@
 		(start 148.041847 109.388)
 		(end 151.4855 109.388)
-		(width 0.21)
+		(width 0.319225)
 		(layer "F.Cu")
 		(net 3)
@@
 		(start 153.0605 109.388)
 		(end 157.023999 109.388)
-		(width 0.21)
+		(width 0.319225)
 		(layer "F.Cu")
 		(net 4)
