File: hardware/programmer/kicad/bwlr1f-prog.kicad_pcb (KiCad board)
At the start: 2 copper layers, 61.2 x 26.1 mm, 35 parts, among them J1 U262-161N-4BVC11, J2 Conn_01x02, J3 Conn_01x02, J4 Conn_01x08, SW1 TL3342F160QG, SW2 TL3342F160QG, U1 USBLC6-2P6, U2 XC6220B331MR-G, U3 CH340E, U4 TXS0102DCUR

Commit message: Added ESD to main board
Parts:
- moved TP2 8.13 mm to (166.4, 71.9)
- moved TP3 4.06 mm to (173.0, 71.9)
- moved TP4 3.30 mm to (176.3, 71.9)
- moved TP5 2.54 mm to (179.6, 71.9)
- moved TP1 2.29 mm to (169.7, 71.9)
- moved TP6 1.78 mm to (182.9, 71.9)
- moved TP7 1.02 mm to (186.2, 71.9)
- moved TP9 0.51 mm to (192.8, 71.9)
- moved TP8 0.25 mm to (189.5, 71.9)
Routing:
- net GND: track 34.3 -> 21.4 mm, vias 114 -> 117
- net +3V0: track 114.0 -> 117.3 mm
- net /TX_A: track 27.4 -> 26.7 mm
- net /RX_A: track 28.1 -> 27.4 mm
Other:
- board text removed: "+3V3 LDO"
- board text removed: "LOGIC SHIFTER"
- board text removed: "UART BRIDGE"

Commit message: Update for Programmer
Parts:
- added D1: ESD5651N, Diode_SMD:D_SOD-882, F.Cu at (191.1, 91.7)
- added D2: ESD5651N, Diode_SMD:D_SOD-882, F.Cu at (187.8, 91.7)
- added D3: ESD5651N, Diode_SMD:D_SOD-882, F.Cu at (184.5, 91.7)
- added D4: ESD5651N, Diode_SMD:D_SOD-882, F.Cu at (181.2, 91.7)
- added D5: ESD5651N, Diode_SMD:D_SOD-882, F.Cu at (177.9, 91.7)
- added D6: ESD5651N, Diode_SMD:D_SOD-882, F.Cu at (174.6, 91.7)
- added D7: ESD5651N, Diode_SMD:D_SOD-882, F.Cu at (168.0, 91.7)
- added D8: ESD5651N, Diode_SMD:D_SOD-882, F.Cu at (171.3, 91.7)
- added G***: LOGO, bwlr1f-prog:TeapotLogo4mm, B.Cu at (184.8, 85.5)
- TP1, TP2, TP3, TP4, TP5, TP6, TP7, TP8, TP9: moved to B.Cu
- moved H3 20.5 mm to (202.3, 92.1)
- moved TP1 19.8 mm to (169.7, 91.7)
- moved TP2 19.8 mm to (166.4, 91.7)
- moved TP3 19.8 mm to (173.0, 91.7)
- moved TP4 19.8 mm to (176.3, 91.7)
- moved TP5 19.8 mm to (179.6, 91.7)
- moved TP6 19.8 mm to (182.9, 91.7)
- moved TP7 19.8 mm to (186.2, 91.7)
- moved TP8 19.8 mm to (189.5, 91.7)
- moved TP9 19.8 mm to (192.8, 91.7)
- moved J4 18.1 mm to (172.6, 79.3), turned to 90 degrees
- moved J3 9.75 mm to (194.2, 79.3), turned to 90 degrees
- moved J2 6.07 mm to (200.5, 79.3), turned to 90 degrees
- moved SW2 3.61 mm to (161.2, 90.3), turned to 90 degrees
- moved SW1 0.63 mm to (154.6, 90.3), turned to -90 degrees
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Connections:
- J2 pad 1: GND -> /RST
- J2 pad 2: /RST -> GND
- J3 pad 1: +3V0 -> /BOOT
- J3 pad 2: /BOOT -> +3V0
- J4 pad 1: GND -> +3V0
- J4 pad 2: /RST -> /SWDIO
- J4 pad 3: /BOOT -> /SWCLK
- J4 pad 4: /RX_A -> /TX_A
- J4 pad 5: /TX_A -> /RX_A
- J4 pad 6: /SWCLK -> /BOOT
- J4 pad 7: /SWDIO -> /RST
- J4 pad 8: +3V0 -> GND
Routing:
- net +3V0: track 117.3 -> 68.5 mm
- net /RX_A: track 27.4 -> 35.7 mm, vias 0 -> 1
- net /RST: track 64.8 -> 72.6 mm, vias 0 -> 1
- net /BOOT: track 64.5 -> 58.9 mm, vias 0 -> 1
- net GND: track 21.4 -> 17.5 mm, vias 117 -> 126
- net +3V3: track 21.4 -> 18.3 mm, vias 0 -> 2
- net /TX_A: track 26.7 -> 29.5 mm, vias 0 -> 1
- net /SWDIO: track 12.7 -> 15.1 mm
- net /SWCLK: track 12.4 -> 14.8 mm
- net +BATT: track 0.00 -> 1.80 mm
- net /TX_B: track 7.71 -> 6.54 mm
- net /RX_B: track 7.70 -> 6.75 mm
Other:
- board text added: "B"
- board text added: "Dimension @User.2"
- board text added: "R"
- board text removed: "RESET"

Commit message: Finish Production File for Programmer Board
Parts:
- F1: value 0.75A -> SMD0805P075TF

Commit message: Revision finish, update production file
Other:
- board text added: "Dimension at User.2"
- board text removed: "Dimension @User.2"
Changed lines of the file:
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@@
 		)
 	)
-	(gr_text "Dimension @User.2"
+	(gr_text "Dimension at User.2"
 		(at 143.909472 97.266001 0)
 		(layer "User.2")

Commit message: clean-up
Other:
- board text added: "PCB3D_BR_bwlr1f_programmer"
- board text added: "PCB3D_TL_bwlr1f_programmer"
- board text added: "Rev. 1"
- board text removed: "08/24"
- board text removed: "REV.A"
Changed lines of the file:
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@@
 	)
 	(paper "A4")
+	(title_block
+		(title "BWLR1F Programmer")
+		(date "2024-08-27")
+		(rev "1")
+		(company "Teapot Laboratories")
+	)
 	(layers
 		(0 "F.Cu" signal)
@@
 		(layer "User.2")
 	)
-	(gr_text "08/24"
-		(at 177.437472 87.487001 -0)
-		(layer "B.SilkS")
-		(effects
-			(font
-				(size 0.8 0.8)
-				(thickness 0.16)
-				(bold yes)
-			)
-			(justify left mirror)
-		)
-	)
-	(gr_text "REV.A"
-		(at 179.723472 87.487001 -0)
+	(gr_text "Rev. 1"
+		(at 179.723472 87.487001 0)
 		(layer "B.SilkS" knockout)
 		(effects
@@
 		)
 	)
+	(gr_text "PCB3D_TL_bwlr1f_programmer"
+		(at 143.723472 68.653001 0)
+		(layer "F.Fab")
+		(effects
+			(font
+				(size 3 3)
+				(thickness 0.15)
+			)
+			(justify left bottom)
+		)
+	)
+	(gr_text "PCB3D_BR_bwlr1f_programmer"
+		(at 205.123472 94.853001 0)
+		(layer "F.Fab")
+		(effects
+			(font
+				(size 3 3)
+				(thickness 0.15)
+			)
+			(justify left bottom)
+		)
+	)
 	(gr_text "Dimension at User.2"
 		(at 143.909472 97.266001 0)
@@
 		)
 		(height -5.619999)
-		(gr_text "1,9000 mm"
+		(gr_text "1.9000 mm"
 			(at 153.053472 65.897001 0)
 			(layer "User.2")
@@
 		)
 		(height 12.414)
-		(gr_text "26,1300 mm"
+		(gr_text "26.1300 mm"
 			(at 214.387472 81.788 90)
 			(layer "User.2")
@@
 		)
 		(height 7.873998)
-		(gr_text "61,2325 mm"
+		(gr_text "61.2325 mm"
 			(at 174.507236 61.699002 0)
 			(layer "User.2")
@@
 		)
 		(height -7.366)
-		(gr_text "2,7940 mm"
+		(gr_text "2.7940 mm"
 			(at 211.219472 93.583001 90)
 			(layer "User.2")
@@
 		)
 		(height 8.382)
-		(gr_text "2,7940 mm"
+		(gr_text "2.7940 mm"
 			(at 203.853472 102.219001 0)
 			(layer "User.2")
@@
 		)
 		(height -4.541663)
-		(gr_text "3,9513 mm"
+		(gr_text "3.9513 mm"
 			(at 141.263386 89.431387 45)
 			(layer "User.2")
