File: hardware/programmer/kicad/bwlr1f-prog.kicad_sch (KiCad schematic)
At the start: 35 parts, among them J1 U262-161N-4BVC11, J2 Conn_01x02, J3 Conn_01x02, J4 Conn_01x08, SW1 TL3342F160QG, SW2 TL3342F160QG, U1 USBLC6-2P6, U2 XC6220B331MR-G, U3 CH340E, U4 TXS0102DCUR

Commit message: Update PCB layout
Other:
- note added: "+3V3 to +3V0 Logic Shifter"
- note added: "Debugging Port"
- note added: "Mounting Hole"
- note added: "Programming Port"
- note added: "Reset and Boot"
- moved on the sheet: H1, H2, H3, J4, R4, TP1, TP2, TP3, TP4, TP5, TP6, TP7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

Commit message: Update for Programmer
Parts:
- added D1, D2, D3, D4, D5, D6, D7, D8: ESD5651N, Diode_SMD:D_SOD-882, symbol Device:D_TVS
Connections:
- net +3V0: now also J3.2 (Pin_2), J4.1 (Pin_1), D8.2 (A2); no longer J3.1 (Pin_1), J4.8 (Pin_8)
- net +BATT: now also D7.2 (A2)
- net BOOT: now also J3.1 (Pin_1), J4.6 (Pin_6), D2.2 (A2); no longer J3.2 (Pin_2), J4.3 (Pin_3)
- net GND: now also J2.2 (Pin_2), J4.8 (Pin_8), D1.1 (A1), D2.1 (A1), D3.1 (A1), D4.1 (A1), D5.1 (A1), D6.1 (A1), D7.1 (A1), D8.1 (A1); no longer J2.1 (Pin_1), J4.1 (Pin_1)
- net RST: now also J2.1 (Pin_1), J4.7 (Pin_7), D1.2 (A2); no longer J2.2 (Pin_2), J4.2 (Pin_2)
- net RX_A: now also J4.5 (Pin_5), D3.2 (A2); no longer J4.4 (Pin_4)
- net SWCLK: now also J4.3 (Pin_3), D5.2 (A2); no longer J4.6 (Pin_6)
- net SWDIO: now also J4.2 (Pin_2), D6.2 (A2); no longer J4.7 (Pin_7)
- net TX_A: now also J4.4 (Pin_4), D4.2 (A2); no longer J4.5 (Pin_5)
Other:
- moved on the sheet: J2, J3, J4, TP1, TP2, TP3, TP4, TP5, TP6, TP7, TP8, TP9

Commit message: Finish Production File for Programmer Board
Parts:
- C1: Distributor (none) -> LCSC; Distributor Link (none) -> https://www.lcsc.com/product-detail/Multilayer-Ceramic-Capa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; Distributor Part Number (none) -> C60133; Manufacturer Part Number (none) -> CC0402KRX7R9BB103; Type (none) -> SMT
- C2: Distributor (none) -> LCSC; Distributor Link (none) -> https://www.lcsc.com/product-detail/Multilayer-Ceramic-Capa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; Distributor Part Number (none) -> C1525; Manufacturer YAGEO -> Samsung Electro-Mechanics; Manufacturer Part Number (none) -> CL05B104KO5NNNC; Type (none) -> SMT
- C3, C4: Distributor (none) -> LCSC; Distributor Link (none) -> https://www.lcsc.com/product-detail/Multilayer-Ceramic-Capa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; Distributor Part Number (none) -> C17024; Manufacturer (none) -> Samsung Electro-Mechanics; Manufacturer Part Number (none) -> CL21A106KPFNNNE; Type (none) -> SMT
- C5: Distributor (none) -> LCSC; Distributor Link (none) -> https://www.lcsc.com/product-detail/Multilayer-Ceramic-Capa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; Distributor Part Number (none) -> C1591; Manufacturer (none) -> Samsung Electro-Mechanics; Manufacturer Part Number (none) -> CL10B104KB8NNNC; Type (none) -> SMT
- C6, C7: Distributor (none) -> LCSC; Distributor Link (none) -> https://www.lcsc.com/product-detail/Multilayer-Ceramic-Capa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; Distributor Part Number (none) -> C1525; Manufacturer (none) -> Samsung Electro-Mechanics; Manufacturer Part Number (none) -> CL05B104KO5NNNC; Type (none) -> SMT
- D1, D2, D3, D4, D5, D6, D7, D8: Type SMD -> SMT
- F1: value 0.75A -> SMD0805P075TF; Distributor (none) -> LCSC; Distributor Link (none) -> https://www.lcsc.com/product-detail/Resettable-Fuses_RUILON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; Distributor Part Number (none) -> C20979; Manufacturer RUILON -> RUILON(Shenzhen Ruilongyuan Elec); Manufacturer Part Number (none) -> SMD0805P075TF; Type (none) -> SMT
- FB1: Distributor (none) -> LCSC; Distributor Link (none) -> https://www.lcsc.com/product-detail/Ferrite-Beads_TDK-MMZ16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; Distributor Part Number (none) -> C97120; Manufacturer Part Number (none) -> MMZ1608B601CTAH0; Type (none) -> SMT
- H1, H2, H3, J2, J3, J4: Distributor (none) -> -; Distributor Link (none) -> -; Distributor Part Number (none) -> -; Manufacturer (none) -> -; Manufacturer Part Number (none) -> -; Type (none) -> THT
- J1: Distributor (none) -> LCSC; Distributor Link (none) -> https://www.lcsc.com/product-detail/USB-Connectors_XKB-Conn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; Distributor Part Number (none) -> C319148; Manufacturer Part Number (none) -> U262-161N-4BVC11; Type (none) -> SMT
- R1, R2, R4: Distributor (none) -> LCSC; Distributor Link (none) -> https://www.lcsc.com/product-detail/Chip-Resistor-Surface-M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; Distributor Part Number (none) -> C25905; Manufacturer (none) -> UNI-ROYAL(Uniroyal Elec); Manufacturer Part Number (none) -> 0402WGF5101TCE; Type (none) -> SMT
- R3: Distributor (none) -> LCSC; Distributor Link (none) -> https://www.lcsc.com/product-detail/Chip-span-style-backgro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; Distributor Part Number (none) -> C25804; Manufacturer (none) -> UNI-ROYAL(Uniroyal Elec); Manufacturer Part Number (none) -> 0603WAF1002T5E; Type (none) -> SMT
- SW1, SW2: Distributor (none) -> LCSC; Distributor Link (none) -> https://www.lcsc.com/product-detail/Tactile-Switches_E-Swit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; Distributor Part Number (none) -> C2886898; Manufacturer Part Number (none) -> TL3342F160QG; Type (none) -> SMT
- TP1, TP2, TP3, TP4, TP5, TP6, TP7, TP8, TP9: Distributor (none) -> Digikey; Distributor Link (none) -> https://www.digikey.com/en/products/detail/preci-dip/90055-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; Distributor Part Number (none) -> 1212-1855-ND; Manufacturer (none) -> Preci-Dip; Manufacturer Part Number (none) -> 90055-AS; Type (none) -> THT
- U1: Distributor (none) -> LCSC; Distributor Link (none) -> https://www.lcsc.com/product-detail/ESD-Protection-Devices_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; Distributor Part Number (none) -> C15999; Manufacturer Part Number (none) -> USBLC6-2P6; Type (none) -> SMT
- U2: Distributor (none) -> LCSC; Distributor Link (none) -> https://www.lcsc.com/product-detail/Linear-Voltage-Regulato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; Distributor Part Number (none) -> C86534; Manufacturer Part Number (none) -> XC6220B331MR-G; Type (none) -> SMT
- U3: Distributor (none) -> LCSC; Distributor Link (none) -> https://www.lcsc.com/product-detail/USB-ICs_WCH-Jiangsu-Qin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; Distributor Part Number (none) -> C99652; Manufacturer Part Number (none) -> CH340E; Type (none) -> SMT
- U4: Distributor (none) -> LCSC; Distributor Link (none) -> https://www.lcsc.com/product-detail/Translators-Level-Shift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; Distributor Part Number (none) -> C53434; Manufacturer (none) -> Texas Instruments; Manufacturer Part Number (none) -> TXS0102DCUR; Type (none) -> SMT
Other:
- moved on the sheet: C6, C7, D1, D2, D3, D4, D5, D6, D7, D8, H1, H2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

Commit message: clean-up
Other:
- company: (none) -> Teapot Laboratories
- title: (none) -> BWLR1F Programmer
Changed lines of the file:
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@@
 	(generator_version "8.0")
 	(paper "A4")
+	(title_block
+		(title "BWLR1F Programmer")
+		(date "2024-08-27")
+		(rev "1")
+		(company "Teapot Laboratories")
+	)
 	(junction
 		(at 256.54 119.38)
